File: hardware/schematics/acorn_digital.kicad_sch (KiCad schematic)
At the start: 28 parts, among them J1 Conn_02x20_Odd_Even, J2 Raspberry_Pi_4, Q1 PN2222A, Q2 PN2222A, U1 WM8731SEDS, U2 ATmega328-P, Y1 16MHz

Commit message: more schematic work
Parts:
- added C10: 47uF, symbol Device:C_Polarized_US
- added C11, C13: 1uF, Capacitor_THT:C_Disc_D4.7mm_W2.5mm_P5.00mm, symbol Device:C_Small
- added C12, C15: 47uF, Capacitor_THT:CP_Radial_D7.5mm_P2.50mm, symbol Device:C_Polarized_US
- added C16, C19, C20, C21, C22, C23: 0.01uF, Capacitor_THT:C_Disc_D4.7mm_W2.5mm_P5.00mm, symbol Device:C_Small
- added C3, C4: 20pF, Capacitor_THT:C_Disc_D4.7mm_W2.5mm_P5.00mm, symbol Device:C_Small
- added C5, C7, C8, C9: 0.1uF, Capacitor_THT:C_Disc_D4.7mm_W2.5mm_P5.00mm, symbol Device:C_Small
- added C?: 0.1 uF, Capacitor_THT:C_Disc_D4.7mm_W2.5mm_P5.00mm, symbol Device:C_Small
- added C?: 470uF, Capacitor_THT:CP_Radial_D7.5mm_P2.50mm, symbol Device:C_Polarized_US
- added D1: 3.6V, symbol Device:D_Zener
- added D2: 3.6V, Diode_THT:D_DO-201AD_P12.70mm_Horizontal, symbol Device:D_Zener
- added D4, D5: 5.2V, Diode_THT:D_DO-201AD_P12.70mm_Horizontal, symbol Device:D_Zener
- added L1: 10uH, Inductor_SMD:L_6.3x6.3_H3, symbol Device:L
- added Q3, Q4: PN2222A, Package_TO_SOT_THT:TO-92_Inline, symbol Transistor_BJT:PN2222A
- added R10, R11, R12, R13, R14, R15: 10K, Resistor_THT:R_Axial_DIN0204_L3.6mm_D1.6mm_P5.08mm_Vertical, symbol Device:R_US
- added R17, R18, R19, R20: 1K, Resistor_THT:R_Axial_DIN0204_L3.6mm_D1.6mm_P5.08mm_Vertical, symbol Device:R_US
- added R5, R6: 4.7K, Resistor_THT:R_Axial_DIN0204_L3.6mm_D1.6mm_P5.08mm_Vertical, symbol Device:R_US
- added Y1: 12.288MHz, Crystal:Crystal_HC18-U_Vertical, symbol Device:Crystal
- J1: footprint (none) -> Connector_PinHeader_1.00mm:PinHeader_2x20_P1.00mm_Vertical
- renumbered C4 to C14, C6 to C17, C5 to C18, C3 to C6, D1 to D3, R8 to R16, R9 to R21, R10 to R22, R11 to R23, R12 to R24, R13 to R25, R14 to R26, R5 to R7, R6 to R8, R7 to R9, Y1 to Y2
Connections:
- net PI RX is gone; now on net PI UART RX: R3.1, U2.3 (PD1)
- net PI TX is gone; now on net PI UART TX: R1.1, U2.2 (PD0)
- net +3.3V: now also U1.1 (DBVDD), U1.27 (DCVDD), C5.1, C7.1, L1.2, R5.1, R6.1
- net +5V: now also J1.1 (Pin_1), J1.2 (Pin_2), C?.1, C?.1
- net GND: now also J1.36 (Pin_36), J1.37 (Pin_37), U1.11 (HPGND), U1.15 (AGND), U1.16 (VMID), U1.21 (MODE), U1.22 (~{CSB}), U1.28 (DGND), C10.2, C16.2, C19.2, C20.2, C21.2, C22.2, C23.2, C3.2, C4.2, C5.2, C7.2, C8.2, C9.2, C?.2, C?.2, D1.2 (A), D2.2 (A), D4.2 (A), D5.2 (A), Q3.1 (E), Q4.1 (E), R10.2, R11.2, R12.2, R13.2, R14.2, R15.2, R18.1, R20.1
- net at U1.10 (RHPOUT): now also C15.1
- net at U1.14 (AVDD): now also U1.8 (HPVDD), C10.1, C8.1, C9.1, L1.1
- net at U1.19 (RLINEIN): now also C13.1
- net at U1.20 (LLINEIN): now also C11.1
- net PI SDA: now reaches U1.23 (SDIN)
- net PI SDA: now also J1.3 (Pin_3), J2.3 (SDA/GPIO2), R5.2
- net PI SCL: now reaches U1.24 (SCLK)
- net PI SCL: now also J1.5 (Pin_5), J2.5 (SCL/GPIO3), R6.2
- net at U1.25 (XTI/MCLK): now also C3.1, Y1.1
- net at U1.26 (XTO): now also C4.1, Y1.2
- net at U1.3 (BCLK): now also J2.12 (GPIO18/PWM0)
- net at U1.4 (DACDAT): now also J2.40 (GPIO21/SCLK1)
- net at U1.5 (DACLRC): now also J2.35 (GPIO19/MISO1), U1.7 (ADCLRC)
- net at U1.6 (ADCDAT): now also J2.38 (GPIO20/MOSI1)
- net at U1.9 (LHPOUT): now also C12.1
- net PTT: now reaches J2.11 (GPIO17)
- net PTT: now also J1.22 (Pin_22), C23.1, Q4.3 (C)
- net ENC2_S: now reaches J2.13 (GPIO27)
- net ENC2_S: now also J1.33 (Pin_33)
- net ENC1_A: now reaches J2.15 (GPIO22)
- net ENC1_A: now also J1.23 (Pin_23)
- net ENC1_B: now reaches J2.16 (GPIO23)
- net ENC1_B: now also J1.25 (Pin_25)
- net ENC1_S: now reaches J2.18 (GPIO24)
- net ENC1_S: now also J1.27 (Pin_27)
- net ENC2_A: now reaches J2.22 (GPIO25)
- net ENC2_A: now also J1.29 (Pin_29)
- net BAND4: now reaches J2.24 (~{CE0}/GPIO8)
- net BAND4: now also J1.17 (Pin_17)
- net BAND3: now reaches J2.26 (~{CE1}/GPIO7)
- net BAND3: now also J1.15 (Pin_15)
- net BAND1: now reaches J2.29 (GCLK1/GPIO5)
- net BAND1: now also J1.11 (Pin_11)
- net BAND2: now reaches J2.31 (GCLK2/GPIO6)
- net BAND2: now also J1.13 (Pin_13)
- net TX: now reaches J2.36 (GPIO16)
- net TX: now also J1.20 (Pin_20)
- net ENC2_B: now reaches J2.37 (GPIO26)
- net ENC2_B: now also J1.31 (Pin_31)
- net AVR1 D6: now reaches J1.10 (Pin_10)
- net AVR1 D6: now also U2.12 (PD6)
- net AVR1 A2: now reaches J1.12 (Pin_12)
- net AVR1 A2: now also U2.25 (PC2)
- net AVR1 A3: now reaches J1.14 (Pin_14)
- net AVR1 A3: now also U2.26 (PC3)
- net AVR1 SDA: now reaches J1.16 (Pin_16)
- net AVR1 SDA: now also U2.27 (PC4)
- net AVR1 SCL: now reaches J1.18 (Pin_18)
- net AVR1 SCL: now also U2.28 (PC5)
- net RF_FORWARD: now reaches J1.19 (Pin_19)
- net RF_FORWARD: now also U2.23 (PC0), C21.1, D4.1 (K)
- net RF_REFL: now reaches J1.21 (Pin_21)
- net RF_REFL: now also U2.24 (PC1), C22.1, D5.1 (K)
- net HEADPHONE: now reaches J1.24 (Pin_24)
- net HEADPHONE: now also R13.1
- net AUDIO MOD: now reaches J1.28 (Pin_28)
- net AUDIO MOD: now also R14.1
- net AUDIO DEMOD: now reaches J1.30 (Pin_30)
- net AUDIO DEMOD: now also R15.1
- net CW PTT: now reaches J1.34 (Pin_34)
- net CW PTT: now also C16.1, Q3.3 (C)
- net PADDLE_LEFT: now reaches J1.38 (Pin_38)
- net PADDLE_LEFT: now also U2.4 (PD2), C19.1
- net MIC: now reaches J1.39 (Pin_39)
- net MIC: now also R12.1
- net AVR1 D9: now reaches J1.4 (Pin_4)
- net AVR1 D9: now also U2.15 (PB1)
- net PADDLE_RIGHT: now reaches J1.40 (Pin_40)
- net PADDLE_RIGHT: now also U2.5 (PD3), C20.1
- net AVR1 D10: now reaches J1.6 (Pin_6)
- net AVR1 D10: now also U2.16 (PB2)
- net PI UART TX: now reaches J1.7 (Pin_7)
- net AVR1 D5: now reaches J1.8 (Pin_8)
- net AVR1 D5: now also U2.11 (PD5)
- net PI UART RX: now reaches J1.9 (Pin_9)
- net at U2.14 (PB0): now also R17.1
- net at U2.6 (PD4): now also R19.2
- net RESET renamed AVR RESET
- new net: C11.2, D2.1 (K)
- new net: C13.2, D1.1 (K)
- new net: Q4.2 (B), R19.1, R20.2
- new net: C12.2, R11.1
- new net: C15.2, R10.1
- new net: Q3.2 (B), R17.2, R18.2
- no-connect marks 104 -> 12
Other:
- moved on the sheet: C17, C18, D3, J1, R1, R16, R2, R21, R22, R23, R24, R25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

Commit message: more schematic work
Parts:
- removed C11, C13: 1uF, Capacitor_THT:C_Disc_D4.7mm_W2.5mm_P5.00mm, symbol Device:C_Small
- removed R12, R13, R14, R15: 10K, Resistor_THT:R_Axial_DIN0204_L3.6mm_D1.6mm_P5.08mm_Vertical, symbol Device:R_US
- added C15, C17, C18, C19, C21: 47uF, Capacitor_THT:CP_Radial_D7.5mm_P2.50mm, symbol Device:C_Polarized_US
- added C20: 100uF, Capacitor_THT:CP_Radial_D7.5mm_P2.50mm, symbol Device:C_Polarized_US
- added C22: 200pF, Capacitor_THT:C_Disc_D4.7mm_W2.5mm_P5.00mm, symbol Device:C_Small
- added C23: 0.01uF, Capacitor_THT:C_Disc_D4.7mm_W2.5mm_P5.00mm, symbol Device:C_Small
- added C24: 10uF, Capacitor_THT:CP_Radial_D7.5mm_P2.50mm, symbol Device:C_Polarized_US
- added D3: 3.6V, Diode_THT:D_DO-201AD_P12.70mm_Horizontal, symbol Device:D_Zener
- added Q1: BS250, Package_TO_SOT_THT:TO-92_Inline, symbol Transistor_FET:BS250
- added Q4: PN2222A, Package_TO_SOT_THT:TO-92_Inline, symbol Transistor_BJT:PN2222A
- added R16, R24, R25: 1K, Resistor_THT:R_Axial_DIN0204_L3.6mm_D1.6mm_P5.08mm_Vertical, symbol Device:R_US
- added R17, R23: 100, Resistor_THT:R_Axial_DIN0204_L3.6mm_D1.6mm_P5.08mm_Vertical, symbol Device:R_US
- added R18: 10K, Resistor_THT:R_Axial_DIN0204_L3.6mm_D1.6mm_P5.08mm_Vertical, symbol Device:R_US
- added R19: 3.3K, Resistor_THT:R_Axial_DIN0204_L3.6mm_D1.6mm_P5.08mm_Vertical, symbol Device:R_US
- added R5: 5K, Resistor_THT:R_Axial_DIN0204_L3.6mm_D1.6mm_P5.08mm_Vertical, symbol Device:R_US
- added R6, R8, R9: 27, Resistor_THT:R_Axial_DIN0204_L3.6mm_D1.6mm_P5.08mm_Vertical, symbol Device:R_US
- added RV1: 10K, Potentiometer_THT:Potentiometer_Piher_PT-6-V_Vertical_Hole, symbol Device:R_Potentiometer_US
- C12: renamed from C10; footprint (none) -> Capacitor_THT:CP_Radial_D7.5mm_P2.50mm
- D1: value 3.6V -> 4V; footprint (none) -> Diode_THT:D_DO-201AD_P12.70mm_Horizontal
- gave numbers to parts that had none: 2
- renumbered C8 to C10, C9 to C11, C12 to C13, C15 to C16, C16 to C25, C17 to C26, C18 to C27, C19 to C28, C20 to C29, C1 to C3, C21 to C30, C22 to C31, C23 to C32, C2 to C4, C3 to C5, C4 to C6, C5 to C7, C6 to C8, C7 to C9, D3 to D4, D4 to D5, D5 to D6, Q1 to Q2, Q2 to Q3, Q3 to Q5, Q4 to Q6, R6 to R10, R7 to R11, R8 to R12, R9 to R13, R10 to R14, R11 to R15, R16 to R20, R17 to R21, R18 to R22, R19 to R26, R20 to R27, R21 to R28, R22 to R29, R23 to R30, R24 to R31, R25 to R32, R26 to R33, R5 to R7
Connections:
- net +5V: now also D1.1 (K), Q1.3 (S), R23.2; no longer C2.1, J1.1 (Pin_1), J1.2 (Pin_2)
- net AUDIO DEMOD: now also C15.2
- net AUDIO MOD: now also C16.2, R14.1
- net GND: now also C19.2, C20.2, C22.2, C23.2, C24.2, D3.2 (A), R17.1, R19.1, R5.2, RV1.3; no longer D1.2 (A)
- net HEADPHONE: now also C13.2, R15.1
- net MIC: now also C21.1, C22.1, R25.1
- net at D2.1 (K): now also U1.19 (RLINEIN), C17.1
- net at U1.20 (LLINEIN): now also C15.1, D3.1 (K)
- net at U1.3 (BCLK): now also R6.1; no longer J2.12 (GPIO18/PWM0)
- net at U1.4 (DACDAT): now also R8.1; no longer J2.40 (GPIO21/SCLK1)
- net at U1.6 (ADCDAT): now also R9.1; no longer J2.38 (GPIO20/MOSI1)
- new net: C21.2, Q4.2 (B), R18.1, R19.2
- new net: J2.40 (GPIO21/SCLK1), R8.2
- new net: C18.1, Q4.3 (C), R16.1
- new net: C18.2, RV1.1
- new net: C19.1, Q4.1 (E), R17.2
- new net: J2.12 (GPIO18/PWM0), R6.2
- new net: C2.1, J1.1 (Pin_1), J1.2 (Pin_2), Q1.1 (D)
- new net: J2.38 (GPIO20/MOSI1), R9.2
- new net: C20.1, C23.1, R16.2, R18.2, R23.1, R24.2
- new net: C24.1, R24.1, R25.2
- new net: D1.2 (A), Q1.2 (G), R5.1
- new net: C17.2, RV1.2
Other:
- moved on the sheet: C1, C2

Commit message: more schematic work
Parts:
- added R13: 27, Resistor_THT:R_Axial_DIN0204_L3.6mm_D1.6mm_P5.08mm_Vertical, symbol Device:R_US
- renumbered R13 to R14, R14 to R15, R15 to R16, R16 to R17, R17 to R18, R18 to R19, R19 to R20, R20 to R21, R21 to R22, R22 to R23, R23 to R24, R24 to R25, R25 to R26, R26 to R27, R27 to R28, R28 to R29, R29 to R30, R30 to R31, R31 to R32, R32 to R33, R33 to R34
Connections:
- net GND: now also R13.1, R13.2

Commit message: testing the wm7831
Parts:
- removed R13: 27, Resistor_THT:R_Axial_DIN0204_L3.6mm_D1.6mm_P5.08mm_Vertical, symbol Device:R_US
- R6, R8, R9: value 27 -> 51
- renumbered R14 to R13, R15 to R14, R16 to R15, R17 to R16, R18 to R17, R19 to R18, R20 to R19, R21 to R20, R22 to R21, R23 to R22, R24 to R23, R25 to R24, R26 to R25, R27 to R26, R28 to R27, R29 to R28, R30 to R29, R31 to R30, R32 to R31, R33 to R32, R34 to R33
