File: hardware/schematics/acorn_rf.kicad_sch (KiCad schematic)
At the start: 0 parts

Commit message: testing the wm7831
Parts:
- added U?: Si5351A-B-GT, Package_SO:MSOP-10_3x3mm_P0.5mm, symbol Oscillator:Si5351A-B-GT
Changed lines of the file:
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@@
 (kicad_sch (version 20211123) (generator eeschema)
   (paper "A4")
+  (symbol (lib_id "Oscillator:Si5351A-B-GT") (at 163.83 67.31 0) (unit 1)
+    (in_bom yes) (on_board yes) (fields_autoplaced)
+    (property "Reference" "U?" (id 0) (at 165.8494 80.01 0)
+      (effects (font (size 1.27 1.27)) (justify left))
+    )
+    (property "Value" "Si5351A-B-GT" (id 1) (at 165.8494 82.55 0)
+      (effects (font (size 1.27 1.27)) (justify left))
+    )
+    (property "Footprint" "Package_SO:MSOP-10_3x3mm_P0.5mm" (id 2) (at 163.83 87.63 0)
+      (effects (font (size 1.27 1.27)) hide)
+    )
+    (property "Datasheet" "https://www.silabs.com/documents/public/data-sheets/Si5351-B.pdf" (id 3) (at 154.94 69.85 0)
+      (effects (font (size 1.27 1.27)) hide)
+    )
+    (pin "1")
+    (pin "10")
+    (pin "2")
+    (pin "3")
+    (pin "4")
+    (pin "5")
+    (pin "6")
+    (pin "7")
+    (pin "8")
+    (pin "9")
+  )
 )

Commit message: WM8731 testing
Parts:
- added C1: 0.1 uF, Capacitor_THT:C_Disc_D4.7mm_W2.5mm_P5.00mm, symbol Device:C_Small
- added J1: Conn_02x20_Odd_Even, Connector_PinSocket_2.54mm:PinSocket_2x20_P2.54mm_Vertical, symbol Connector_Generic:Conn_02x20_Odd_Even
- added Q1, Q2: BSS138, Package_TO_SOT_SMD:SOT-23, symbol Transistor_FET:BSS138
- added R1, R2, R3, R4: 10K, Resistor_THT:R_Axial_DIN0204_L3.6mm_D1.6mm_P5.08mm_Vertical, symbol Device:R_US
- added Y1: 25MHz, Crystal:Crystal_HC18-U_Vertical, symbol Device:Crystal
- gave numbers to parts that had none: 1
Connections:
- net +3.3V: now reaches U1.1 (VDD)
- net +3.3V: now also U1.7 (VDDO), C1.1, R3.2, R4.2
- net at U1.2 (XA): now also Y1.1
- net at U1.3 (XB): now also Y1.2
- net at U1.4 (SCL): now also Q1.3 (D), R3.1
- net at U1.5 (SDA): now also Q2.3 (D), R4.1
- net GND: now reaches U1.8 (GND)
- net GND: now also C1.2, J1.36 (Pin_36), J1.37 (Pin_37)
- new net +5V: J1.1 (Pin_1), J1.2 (Pin_2), Q1.1 (G), Q2.1 (G), R1.2, R2.2
- new net AUDIO DEMOD: J1.30 (Pin_30)
- new net AUDIO MOD: J1.28 (Pin_28)
- new net AVR1 A2: J1.12 (Pin_12)
- new net AVR1 A3: J1.14 (Pin_14)
- new net AVR1 D10: J1.6 (Pin_6)
- new net AVR1 D5: J1.8 (Pin_8)
- new net AVR1 D6: J1.10 (Pin_10)
- new net AVR1 D9: J1.4 (Pin_4)
- new net AVR1 SCL: J1.18 (Pin_18), Q1.2 (S), R1.1
- new net AVR1 SDA: J1.16 (Pin_16), Q2.2 (S), R2.1
- new net BAND1: J1.11 (Pin_11)
- new net BAND2: J1.13 (Pin_13)
- new net BAND3: J1.15 (Pin_15)
- new net BAND4: J1.17 (Pin_17)
- new net CW PTT: J1.34 (Pin_34)
- new net ENC1_A: J1.23 (Pin_23)
- new net ENC1_B: J1.25 (Pin_25)
- new net ENC1_S: J1.27 (Pin_27)
- new net ENC2_A: J1.29 (Pin_29)
- new net ENC2_B: J1.31 (Pin_31)
- new net ENC2_S: J1.33 (Pin_33)
- new net HEADPHONE: J1.24 (Pin_24)
- new net MIC: J1.39 (Pin_39)
- new net PADDLE_LEFT: J1.38 (Pin_38)
- new net PADDLE_RIGHT: J1.40 (Pin_40)
- new net PI SCL: J1.5 (Pin_5)
- new net PI SDA: J1.3 (Pin_3)
- new net PI UART RX: J1.9 (Pin_9)
- new net PI UART TX: J1.7 (Pin_7)
- new net PTT: J1.22 (Pin_22)
- new net RF_FORWARD: J1.19 (Pin_19)
- new net RF_REFL: J1.21 (Pin_21)
- new net TX: J1.20 (Pin_20)
- no-connect marks 0 -> 6

Commit message: more schematic work
Parts:
- added C2: 20pF, symbol Device:C_Trim_Small
- added C3: 100pF, Capacitor_THT:C_Disc_D4.7mm_W2.5mm_P5.00mm, symbol Device:C_Small
- added C4, C5: 0.1 uF, Capacitor_THT:C_Disc_D4.7mm_W2.5mm_P5.00mm, symbol Device:C_Small
- added D1, D2: 1N5711, Diode_THT:D_DO-35_SOD27_P7.62mm_Horizontal, symbol Diode:1N5711
- added R10, R11, R12, R13, R7, R8, R9: 10K, Resistor_THT:R_Axial_DIN0204_L3.6mm_D1.6mm_P5.08mm_Vertical, symbol Device:R_US
- added R5: 3.3K, Resistor_THT:R_Axial_DIN0204_L3.6mm_D1.6mm_P5.08mm_Vertical, symbol Device:R_US
- added R6: 150, Resistor_THT:R_Axial_DIN0204_L3.6mm_D1.6mm_P5.08mm_Vertical, symbol Device:R_US
- added T1: SWR, symbol Device:L
- added T2: SWR, symbol Device:L_Coupled_Small_1243
Connections:
- net GND: now also C3.2, C4.2, C5.2, R10.1, R11.1, R12.1, R13.1, R5.1, R7.2, R8.2, R9.1
- net RF_FORWARD: now also C4.1, D1.1 (K), R7.1
- net RF_REFL: now also C5.1, D2.1 (K), R13.2
- net LO: now reaches U1.10 (CLK0)
- net LO: now also R9.2
- net LO2: now reaches U1.6 (CLK2)
- net LO2: now also R11.2
- net BFO: now reaches U1.9 (CLK1)
- net BFO: now also R10.2
- new net: D1.2 (A), R6.1, T2.1
- new net: D2.2 (A), R6.2, T2.3
- new net: C2.2, C3.1, R5.2, T2.2, T2.4
- new net RF IN: C2.1, R8.1, T1.2
- new net RF OUT: R12.2, T1.1
- no-connect marks 6 -> 3
