File: hardware/schematics/acorn_rf.kicad_sch (KiCad schematic)
At the start: 27 parts, among them J1 Conn_02x20_Odd_Even, Q1 BSS138, Q2 BSS138, T1 SWR, T2 SWR, U1 Si5351A-B-GT, Y1 25MHz

Commit message: 2023.03.14 1306 work
Parts:
- removed C2: 20pF, symbol Device:C_Trim_Small
- removed C3: 100pF, Capacitor_THT:C_Disc_D4.7mm_W2.5mm_P5.00mm, symbol Device:C_Small
- removed C4, C5: 0.1 uF, Capacitor_THT:C_Disc_D4.7mm_W2.5mm_P5.00mm, symbol Device:C_Small
- removed D1, D2: 1N5711, Diode_THT:D_DO-35_SOD27_P7.62mm_Horizontal, symbol Diode:1N5711
- removed R5: 3.3K, Resistor_THT:R_Axial_DIN0204_L3.6mm_D1.6mm_P5.08mm_Vertical, symbol Device:R_US
- removed R6: 150, Resistor_THT:R_Axial_DIN0204_L3.6mm_D1.6mm_P5.08mm_Vertical, symbol Device:R_US
- removed T1: SWR, symbol Device:L
- removed T2: SWR, symbol Device:L_Coupled_Small_1243
- added C31, C34, C35, C36: 200pF, Capacitor_THT:C_Disc_D4.7mm_W2.5mm_P5.00mm, symbol Device:C_Small
- added C32, C33: 100pF, Capacitor_THT:C_Disc_D4.7mm_W2.5mm_P5.00mm, symbol Device:C_Small
- added D8, D9: BAT54S, Package_TO_SOT_SMD:SOT-23, symbol Diode:BAT54S
- added L1, L2, L3: T30-6 10T, symbol Device:L
- added L4, L5: T30-6 9T, symbol Device:L
- added TR1, TR3: TRANSF3, symbol Transformer:TRANSF3
- renumbered C1 to C26, J1 to J6, Q1 to Q6, Q2 to Q7, R1 to R29, R2 to R30, R3 to R31, R4 to R32, R7 to R33, R8 to R34, R9 to R35, R10 to R36, R11 to R37, R12 to R38, R13 to R39, U1 to U2, Y1 to Y2
Connections:
- net GND: now also C31.2, C32.2, C33.2, C34.2, C35.2, C36.2, TR1.2, TR1.4, TR1.5
- new net: C35.1, L1.1, L2.2
- new net: C34.1, L1.2, L3.1
- new net: C36.1, L2.1, L5.2
- new net: C33.1, L5.1
- new net: D8.3 (COM), TR3.3
- new net: TR3.4, TR3.5
- new net: D9.3 (COM), TR3.6
- new net: C31.1, L3.2, L4.1
- new net: D8.1 (A), D9.2 (K), TR1.3
- new net: D8.2 (K), D9.1 (A), TR1.6
- new net: C32.1, L4.2
Other:
- moved on the sheet: C26, Q6, Q7, R29, R30, R31, R32, U2, Y2

Commit message: 2023.03.14 2250 work
Parts:
- added C37, C38, C40, C41: 33pF, Capacitor_THT:C_Disc_D4.7mm_W2.5mm_P5.00mm, symbol Device:C_Small
- added C39, C46, C54: 39pF, Capacitor_THT:C_Disc_D4.7mm_W2.5mm_P5.00mm, symbol Device:C_Small
- added C42, C43: 18pF, Capacitor_THT:C_Disc_D4.7mm_W2.5mm_P5.00mm, symbol Device:C_Small
- added C44, C45, C48, C53: .01, Capacitor_THT:C_Disc_D4.7mm_W2.5mm_P5.00mm, symbol Device:C_Small
- added C47, C52: 75pF, Capacitor_THT:C_Disc_D4.7mm_W2.5mm_P5.00mm, symbol Device:C_Small
- added C49, C51: 20pF, Capacitor_THT:C_Disc_D4.7mm_W2.5mm_P5.00mm, symbol Device:C_Small
- added C50: 82pF, Capacitor_THT:C_Disc_D4.7mm_W2.5mm_P5.00mm, symbol Device:C_Small
- added D10, D11, D12, D13, D14, D15, D16, D17, D18, D19, D20, D21: 1N4148, Diode_THT:D_DO-35_SOD27_P7.62mm_Horizontal, symbol Diode:1N4148
- added L10, L11, L12, L13, L14, L18, L19, L9: ?mH, symbol Device:L
- added L15, L16, L17, L6, L7, L8: 0.1uH, symbol Device:L
- added R5 (x2): 5K, Resistor_THT:R_Axial_DIN0204_L3.6mm_D1.6mm_P5.08mm_Vertical, symbol Device:R_US
Connections:
- net BAND1: now also D16.2 (A)
- net BAND2: now also D17.2 (A)
- net BAND3: now also D14.2 (A)
- net BAND4: now also D15.2 (A)
- net GND: now also C38.2, C39.2, C40.2, C44.2, C45.2, C47.2, C48.2, C50.2, C52.2, C53.2, L10.1, L13.1, L15.1, L16.1, L17.1, L19.1, L6.1, L7.1, L8.1, L9.1
- net LO: now also C41.1, C54.1; no longer U2.10 (CLK0)
- net at TR1.1: now also C32.1, L4.2
- new net: C47.1, C49.2, D19.1 (K), L15.2
- new net: D18.2 (A), D19.2 (A), L14.1
- new net: C48.1, C53.1, L14.2, L18.2, R5.2
- new net: C51.1, C52.1, D20.1 (K), L17.2
- new net: D20.2 (A), D21.2 (A), L18.1
- new net: D14.1 (K), D15.1 (K), R5.1
- new net: C44.1, C45.1, L11.2, L12.2, R5.2
- new net: C41.2, D12.1 (K), L10.2
- new net: C37.1, D11.1 (K), L9.2
- new net: C37.2, C46.2, U2.10 (CLK0)
- new net: C40.1, C42.1, D13.1 (K), L8.2
- new net: C49.1, C50.1, C51.2, L16.2
- new net: C39.1, C42.2, C43.1, L7.2
- new net: C38.1, C43.2, D10.1 (K), L6.2
- new net: D16.1 (K), D17.1 (K), R5.1
- new net: C46.1, D18.1 (K), L13.2
- new net: D12.2 (A), D13.2 (A), L11.1
- new net: C54.2, D21.1 (K), L19.2
- new net: D10.2 (A), D11.2 (A), L12.1
Other:
- moved on the sheet: D8, D9, TR1, TR3
