File: hardware/schematics/acorn.kicad_sch (KiCad schematic)
At the start: 12 parts, among them J1 Raspberry_Pi_4, U1 ATmega328-P

Commit message: more schematic work
Parts:
- removed C1: 0.1uF, Capacitor_THT:C_Disc_D4.7mm_W2.5mm_P5.00mm, symbol Device:C_Small
- removed C2: 0.1 uF, Capacitor_THT:C_Disc_D4.7mm_W2.5mm_P5.00mm, symbol Device:C_Small
- removed D1: LED, LED_THT:LED_D4.0mm, symbol Device:LED
- removed J1: Raspberry_Pi_4, Connector_PinSocket_2.54mm:PinSocket_2x20_P2.54mm_Vertical, symbol Connector:Raspberry_Pi_2_3
- removed R1, R3, R5, R7: 1K, Resistor_THT:R_Axial_DIN0204_L3.6mm_D1.6mm_P5.08mm_Vertical, symbol Device:R_US
- removed R2, R4, R6: 2K, Resistor_THT:R_Axial_DIN0204_L3.6mm_D1.6mm_P5.08mm_Vertical, symbol Device:R_US
- removed U1: ATmega328-P, Package_DIP:DIP-28_W7.62mm, symbol MCU_Microchip_ATmega:ATmega328-P
Connections:
- no-connect marks 44 -> 0
Other:
- added sheet Digital (acorn_digital.kicad_sch)
- added sheet RF (acorn_rf.kicad_sch)

Commit message: WM8731 testing
Other:
- sheet Digital renamed Control
- sheet Control: file acorn_digital.kicad_sch -> acorn_control.kicad_sch
