File: hardware/schematics/acorn.kicad_sch (KiCad schematic)
At the start: 0 parts

Commit message: 2023.03.14 1306 work
Other:
- added sheet TX - TR (TX-TR.kicad_sch)
Changed lines of the file:
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@@
     (instances
       (project "acorn"
-        (path "/bbe2252c-acad-49f6-93c3-633539ee972c" (page "3"))
+        (path "/bbe2252c-acad-49f6-93c3-633539ee972c" (page "2"))
+      )
+    )
+  )
+  (sheet (at 36.83 111.76) (size 101.6 50.8) (fields_autoplaced)
+    (stroke (width 0.1524) (type solid))
+    (fill (color 0 0 0 0.0000))
+    (property "Sheetname" "TX - TR" (at 36.83 111.0484 0)
+      (effects (font (size 1.27 1.27)) (justify left bottom))
+    )
+    (property "Sheetfile" "TX-TR.kicad_sch" (at 36.83 163.1446 0)
+      (effects (font (size 1.27 1.27)) (justify left top))
+    )
+    (instances
+      (project "acorn"
+        (path "/bbe2252c-acad-49f6-93c3-633539ee972c" (page "4"))
       )
     )
@@
     (instances
       (project "acorn"
-        (path "/bbe2252c-acad-49f6-93c3-633539ee972c" (page "2"))
+        (path "/bbe2252c-acad-49f6-93c3-633539ee972c" (page "3"))
       )
     )
