File: hardware/schematics/acorn_control.kicad_sch (KiCad schematic)
At the start: 82 parts, among them J2 Conn_02x20_Odd_Even, J3 Raspberry_Pi_4, Q3 PN2222A, Q4 PN2222A, Q5 PN2222A, Q6 PN2222A, Q7 PN2222A, U2 WM8731SEDS, U3 ATmega328-P, Y2 12.288MHz, Y3 16MHz

Commit message: working on tcpserver
Parts:
- added R23: 10K, Resistor_THT:R_Axial_DIN0204_L3.6mm_D1.6mm_P5.08mm_Vertical, symbol Device:R_US
- R24: renamed from R23; value 1K -> 10K
- R25: renamed from R24; value 1K -> 10K
- renumbered C14 to C13, C15 to C14, C13 to C15, R25 to R26, R26 to R27, R27 to R28, R28 to R29, R29 to R30, R30 to R31, R31 to R32, R32 to R33, R33 to R34, R34 to R35, R35 to R36, R36 to R37, R37 to R38, R38 to R39, R39 to R40, R40 to R41, R41 to R42, R42 to R43, R43 to R44, R44 to R45, R45 to R46
Connections:
- net +3.3V: now also R23.1
- net at J3.7 (GCLK0/GPIO4), R24.2: now also R23.2
Other:
- moved on the sheet: C15, Q3, Q4, R24, R25, R26

Commit message: 20230128 work
Connections:
- net BAND_HF: now reaches J3.32 (PWM0/GPIO12)
- net BAND_HF: now also J2.35 (Pin_35)
- no-connect marks 12 -> 10
Changed lines of the file:
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@@
   (no_connect (at 151.13 127))
   (no_connect (at 151.13 129.54))
-  (no_connect (at 45.72 177.8))
   (no_connect (at 115.57 144.78))
   (no_connect (at 151.13 142.24))
-  (no_connect (at 99.06 85.09))
   (no_connect (at 58.42 165.1))
   (no_connect (at 99.06 46.99))
@@
     (stroke (width 0) (type default) (color 0 0 0 0))
   )
+  (wire (pts (xy 99.06 85.09) (xy 102.87 85.09))
+    (stroke (width 0) (type default) (color 0 0 0 0))
+  )
   (wire (pts (xy 134.62 59.69) (xy 133.35 59.69))
     (stroke (width 0) (type default) (color 0 0 0 0))
@@
     )
   )
+  (global_label "BAND_HF" (shape output) (at 45.72 177.8 180) (fields_autoplaced)
+    (effects (font (size 1.27 1.27)) (justify right))
+    (property "Intersheet References" "${INTERSHEET_REFS}" (id 0) (at 34.9612 177.7206 0)
+      (effects (font (size 1.27 1.27)) (justify right) hide)
+    )
+  )
   (global_label "ENC2_A" (shape input) (at 45.72 170.18 180) (fields_autoplaced)
     (effects (font (size 1.27 1.27)) (justify right))
@@
       (effects (font (size 1.27 1.27)) (justify left) hide)
     )
+  )
+  (global_label "BAND_HF" (shape output) (at 102.87 85.09 0) (fields_autoplaced)
+    (effects (font (size 1.27 1.27)) (justify left))
+    (property "Intersheet References" "${INTERSHEET_REFS}" (id 0) (at 113.6288 85.0106 0)
+      (effects (font (size 1.27 1.27)) (justify left) hide)
+    )
