File: hardware/schematics/acorn_control.kicad_sch (KiCad schematic)
At the start: 83 parts, among them J2 Conn_02x20_Odd_Even, J3 Raspberry_Pi_4, Q3 PN2222A, Q4 PN2222A, Q5 PN2222A, Q6 PN2222A, Q7 PN2222A, U2 WM8731SEDS, U3 ATmega328-P, Y2 12.288MHz, Y3 16MHz

Commit message: 2023.03.13 1736 work
Parts:
- removed C10, C11: 20pF, Capacitor_THT:C_Disc_D4.7mm_W2.5mm_P5.00mm, symbol Device:C_Small
- removed C12, C13, C14, C16: 0.1uF, Capacitor_THT:C_Disc_D4.7mm_W2.5mm_P5.00mm, symbol Device:C_Small
- removed C17: 47uF, Capacitor_THT:CP_Radial_D7.5mm_P2.50mm, symbol Device:C_Polarized_US
- removed L1: 10uH, Inductor_SMD:L_6.3x6.3_H3, symbol Device:L
- removed R18, R19: 1K, Resistor_THT:R_Axial_DIN0204_L3.6mm_D1.6mm_P5.08mm_Vertical, symbol Device:R_US
- removed R20, R21, R22: 51, Resistor_THT:R_Axial_DIN0204_L3.6mm_D1.6mm_P5.08mm_Vertical, symbol Device:R_US
- removed U2: WM8731SEDS, Package_SO:SSOP-28_5.3x10.2mm_P0.65mm, symbol Audio:WM8731SEDS
- removed Y2: 12.288MHz, Crystal:Crystal_HC18-U_Vertical, symbol Device:Crystal
- added J4: Codec Hat Connector, Connector_PinHeader_1.00mm:PinHeader_2x20_P1.00mm_Vertical, symbol Connector_Generic:Conn_02x20_Odd_Even
- J2: value Conn_02x20_Odd_Even -> RF Board
Connections:
- no-connect marks 10 -> 5

Commit message: 2023.03.13 1848 work
Parts:
- added J5: Codec Audio Out, Connector_PinHeader_2.54mm:PinHeader_1x04_P2.54mm_Vertical, symbol Connector:Conn_01x04_Pin
- added J6: Codec Audio In, Connector_PinHeader_2.54mm:PinHeader_1x04_P2.54mm_Vertical, symbol Connector:Conn_01x04_Pin
Connections:
- net +3.3V: now also J4.1 (Pin_1), J4.17 (Pin_17)
- net +5V: now also J4.2 (Pin_2), J4.4 (Pin_4)
- net BAND1: now also J4.29 (Pin_29)
- net BAND2: now also J4.31 (Pin_31)
- net BAND3: now also J4.26 (Pin_26)
- net BAND4: now also J4.24 (Pin_24)
- net BAND_HF: now also J4.32 (Pin_32)
- net ENC1_A: now also J4.15 (Pin_15)
- net ENC1_B: now also J4.16 (Pin_16)
- net ENC1_S: now also J4.18 (Pin_18)
- net ENC2_A: now also J4.22 (Pin_22)
- net ENC2_B: now also J4.37 (Pin_37)
- net ENC2_S: now also J4.13 (Pin_13)
- net GND: now also J4.14 (Pin_14), J4.20 (Pin_20), J4.25 (Pin_25), J4.30 (Pin_30), J4.34 (Pin_34), J4.39 (Pin_39), J4.6 (Pin_6), J4.9 (Pin_9), J5.2 (Pin_2), J5.4 (Pin_4), J6.2 (Pin_2), J6.4 (Pin_4)
- net MISO: now also J4.21 (Pin_21)
- net MOSI: now also J4.19 (Pin_19)
- net PI SCL: now also J4.5 (Pin_5)
- net PI SDA: now also J4.3 (Pin_3)
- net PTT: now also J4.11 (Pin_11)
- net SCLK: now also J4.23 (Pin_23)
- net TX: now also J4.36 (Pin_36)
- net GPIO14: now reaches J3.8 (GPIO14/TXD), R14.2, R15.1
- net GPIO14: now also J4.8 (Pin_8)
- net at C21.1: now also J5.3 (Pin_3)
- net GPIO4: now reaches J3.7 (GCLK0/GPIO4), R23.2, R24.2
- net GPIO4: now also J4.7 (Pin_7)
- net GPIO15: now reaches J3.10 (GPIO15/RXD), R16.2, R17.1
- net GPIO15: now also J4.10 (Pin_10)
- net GPIO18: now reaches J3.12 (GPIO18/PWM0)
- net GPIO18: now also J4.12 (Pin_12)
- net GPIO0: now reaches J3.27 (ID_SD/GPIO0)
- net GPIO0: now also J4.27 (Pin_27)
- net GPIO1: now reaches J3.28 (ID_SC/GPIO1)
- net GPIO1: now also J4.28 (Pin_28)
- net GPIO13: now reaches J3.33 (PWM1/GPIO13)
- net GPIO13: now also J4.33 (Pin_33)
- net GPIO19: now reaches J3.35 (GPIO19/MISO1)
- net GPIO19: now also J4.35 (Pin_35)
- net GPIO20: now reaches J3.38 (GPIO20/MOSI1)
- net GPIO20: now also J4.38 (Pin_38)
- net GPIO21: now reaches J3.40 (GPIO21/SCLK1)
- net GPIO21: now also J4.40 (Pin_40)
- net at C20.1, D4.1 (K): now also C22.1, D3.1 (K), J6.1 (Pin_1), J6.3 (Pin_3)
- net at C18.1: now also J5.1 (Pin_1)
- no-connect marks 5 -> 2
Other:
- moved on the sheet: C22, D3

Commit message: 2023.03.14 1306 work
Parts:
- renumbered C6 to C1, C22 to C10, C23 to C11, C24 to C12, C25 to C13, C26 to C14, C27 to C15, C28 to C16, C29 to C17, C30 to C18, C31 to C19, C7 to C2, C32 to C20, C33 to C21, C34 to C22, C35 to C23, C36 to C24, C37 to C25, C8 to C3, C9 to C4, C15 to C5, C18 to C6, C19 to C7, C20 to C8, C21 to C9, D3 to D1, D4 to D2, D5 to D3, D6 to D4, D7 to D5, J2 to J1, J3 to J2, J4 to J3, J5 to J4, J6 to J5, Q3 to Q1, Q4 to Q2, Q5 to Q3, Q6 to Q4, Q7 to Q5, R14 to R1, R28 to R10, R29 to R11, R30 to R12, R31 to R13, R32 to R14, R33 to R15, R34 to R16, R35 to R17, R36 to R18, R37 to R19, R15 to R2, R38 to R20, R39 to R21, R40 to R22, R41 to R23, R42 to R24, R43 to R25, R44 to R26, R45 to R27, R46 to R28, R16 to R3, R17 to R4, R23 to R5, R24 to R6, R25 to R7, R26 to R8, R27 to R9, U3 to U1, Y3 to Y1
